Commit message: master

File: launch/include/config/robot.urdf.xacro (robot description, xacro)
@@ -7,4 +7,10 @@
     <parent link="base_link"/>
     <child link="chassis_link" />
+    <origin xyz="0 0 0" rpy="0 0 0" />
+  </joint>
+  <link name="horizon_frame"> </link>
+  <joint name="horizon_joint" type="fixed">
+    <parent link="chassis_link" />
+    <child link="horizon_frame" />
     <origin xyz="0 0 0" rpy="0 0 0" />
   </joint>
